File: hardware/uob-hep-pc068a-cryosub/mosfet_diff_pair_01.sch (KiCad schematic (older format))
At the start: 13 parts, among them Q1 BSS127S, Q2 BSS127S

Commit message: Tuning simulation to change on/off temperature. Then making the resulting changes to BoM
Parts:
- R1, R7: value 6.6k -> 8.2k
- R2: value 10k -> 12k
Other:
- note added: "Switch at 20 deg C"
Changed lines of the file:
@@
 P 6750 3400
 F 0 "R7" H 6820 3445 50  0000 L CNN
-F 1 "6.6k" H 6820 3355 50  0000 L CNN
+F 1 "8.2k" H 6820 3355 50  0000 L CNN
 F 2 "" V 6680 3400 50  0001 C CNN
 F 3 "~" H 6750 3400 50  0001 C CNN
@@
 P 3350 3400
 F 0 "R1" H 3420 3445 50  0000 L CNN
-F 1 "6.6k" H 3420 3355 50  0000 L CNN
+F 1 "8.2k" H 3420 3355 50  0000 L CNN
 F 2 "" V 3280 3400 50  0001 C CNN
 F 3 "~" H 3350 3400 50  0001 C CNN
@@
 P 3350 4400
 F 0 "R2" H 3420 4445 50  0000 L CNN
-F 1 "10k" H 3420 4355 50  0000 L CNN
+F 1 "12k" H 3420 4355 50  0000 L CNN
 F 2 "" V 3280 4400 50  0001 C CNN
 F 3 "~" H 3350 4400 50  0001 C CNN
@@
 Wire Wire Line
 	6750 4550 6750 4850
+Text Notes 1450 5350 0    50   ~ 0
+Switch at 20 deg C
 $EndSCHEMATC
