File: hardware/uob-hep-pc068a-cryosub/mosfet_diff_pair_load_switch_on_when_warm_01.sch (KiCad schematic (older format))
At the start: 13 parts, among them Q1 BSS127S, Q2 BSS127S

Commit message: Commiting progress so far
Parts:
- added C1: 30nF, Capacitor_SMD:C_0201_0603Metric_Pad0.64x0.40mm_HandSolder, symbol Device:C
- added C2: 1uF, Capacitor_SMD:C_0805_2012Metric_Pad1.18x1.45mm_HandSolder, symbol Device:C
- added Q3: FDD306P, Package_TO_SOT_SMD:TO-252-3_TabPin2, symbol Device:Q_PMOS_GDS
- added R10: 1k, Resistor_SMD:R_0603_1608Metric_Pad0.98x0.95mm_HandSolder, symbol Device:R
- added R6: 5, symbol Device:R
- R1, R2, R3, R4, R5, R7: footprint (none) -> Resistor_SMD:R_0603_1608Metric_Pad0.98x0.95mm_HandSolder
- R8, R9: value 600k -> 20k; footprint (none) -> Resistor_SMD:R_0603_1608Metric_Pad0.98x0.95mm_HandSolder
- TH1: footprint (none) -> Resistor_SMD:R_0805_2012Metric_Pad1.20x1.40mm_HandSolder
Connections:
- net 0: now also C2.2, R6.2
- net 5V0: now also Q3.3 (S)
- net VD1: now also R10.2
- new net: C1.2, Q3.1 (G), R10.1
- new net vload: C1.1, C2.1, Q3.2 (D), R6.1
Other:
- note added: "+pspice \n.TEMP 27\n.CONTROL \nOPTIONS ABSTOL=1nA CHGTOL=1pC ITL1=150 ITL2=150 ITL4=500 RELTOL=0.011\nset filetype=ascii\nset wr_vecnames\nset wr_singlescale\nwrdata tmp.txt V("/vd1") V("/vd2") V("/vcont") V("/vload")\n.ENDC\n* .IC V(/vd2)=2.0 V(/vd1)=4.5"
- note removed: "+pspice \n.TEMP 27\n.CONTROL \nOPTIONS ABSTOL=1nA CHGTOL=1pC ITL1=150 ITL2=150 ITL4=500 RELTOL=0.011\nset filetype=ascii\nset wr_vecnames\nset wr_singlescale\nwrdata tmp.txt V("/vd1") V("/vd2") V("/vcont")\n.ENDC\n* .IC V(/vd2)=2.0 V(/vd1)=4.5"
Changed lines of the file:
@@
 encoding utf-8
 Sheet 1 1
-Title ""
-Date ""
-Rev ""
-Comp ""
-Comment1 ""
+Title "Thermal Switch - On when warm"
+Date "2021-04-12"
+Rev "v0.1"
+Comp "University of Bristol"
+Comment1 "Copyright - CERN-OHL-S"
 Comment2 ""
 Comment3 ""
@@
 F 0 "R7" H 6820 3445 50  0000 L CNN
 F 1 "6.6k" H 6820 3355 50  0000 L CNN
-F 2 "" V 6680 3400 50  0001 C CNN
+F 2 "Resistor_SMD:R_0603_1608Metric_Pad0.98x0.95mm_HandSolder" V 6680 3400 50  0001 C CNN
 F 3 "~" H 6750 3400 50  0001 C CNN
 	1    6750 3400
@@
 Wire Wire Line
 	2450 4500 2450 4850
-Text Notes 2850 2650 2    50   ~ 0
-+pspice \n.TEMP 27\n.CONTROL \nOPTIONS ABSTOL=1nA CHGTOL=1pC ITL1=150 ITL2=150 ITL4=500 RELTOL=0.011\nset filetype=ascii\nset wr_vecnames\nset wr_singlescale\nwrdata tmp.txt V("/vd1") V("/vd2") V("/vcont")\n.ENDC\n* .IC V(/vd2)=2.0  V(/vd1)=4.5
+Text Notes 3800 1700 2    50   ~ 0
++pspice \n.TEMP 27\n.CONTROL \nOPTIONS ABSTOL=1nA CHGTOL=1pC ITL1=150 ITL2=150 ITL4=500 RELTOL=0.011\nset filetype=ascii\nset wr_vecnames\nset wr_singlescale\nwrdata tmp.txt V("/vd1") V("/vd2") V("/vcont") V("/vload")\n.ENDC\n* .IC V(/vd2)=2.0  V(/vd1)=4.5
 Wire Wire Line
 	5550 3850 5800 3850
@@
 F 0 "R5" H 5320 3245 50  0000 L CNN
 F 1 "4.7k" H 5320 3155 50  0000 L CNN
-F 2 "" V 5180 3200 50  0001 C CNN
+F 2 "Resistor_SMD:R_0603_1608Metric_Pad0.98x0.95mm_HandSolder" V 5180 3200 50  0001 C CNN
 F 3 "~" H 5250 3200 50  0001 C CNN
 	1    5250 3200
@@
 P 4900 3450
 F 0 "R9" V 5106 3450 50  0000 C CNN
-F 1 "600k" V 5015 3450 50  0000 C CNN
-F 2 "" V 4830 3450 50  0001 C CNN
+F 1 "20k" V 5015 3450 50  0000 C CNN
+F 2 "Resistor_SMD:R_0603_1608Metric_Pad0.98x0.95mm_HandSolder" V 4830 3450 50  0001 C CNN
 F 3 "~" H 4900 3450 50  0001 C CNN
 	1    4900 3450
@@
 F 0 "R3" H 4020 3195 50  0000 L CNN
 F 1 "4.7k" H 4020 3105 50  0000 L CNN
-F 2 "" V 3880 3150 50  0001 C CNN
+F 2 "Resistor_SMD:R_0603_1608Metric_Pad0.98x0.95mm_HandSolder" V 3880 3150 50  0001 C CNN
 F 3 "~" H 3950 3150 50  0001 C CNN
 	1    3950 3150
@@
 P 4300 3600
 F 0 "R8" V 4400 3600 50  0000 C CNN
-F 1 "600k" V 4200 3600 50  0000 C CNN
-F 2 "" V 4230 3600 50  0001 C CNN
+F 1 "20k" V 4200 3600 50  0000 C CNN
+F 2 "Resistor_SMD:R_0603_1608Metric_Pad0.98x0.95mm_HandSolder" V 4230 3600 50  0001 C CNN
 F 3 "~" H 4300 3600 50  0001 C CNN
 	1    4300 3600
@@
 F 0 "R1" H 3420 3445 50  0000 L CNN
 F 1 "6.6k" H 3420 3355 50  0000 L CNN
-F 2 "" V 3280 3400 50  0001 C CNN
+F 2 "Resistor_SMD:R_0603_1608Metric_Pad0.98x0.95mm_HandSolder" V 3280 3400 50  0001 C CNN
 F 3 "~" H 3350 3400 50  0001 C CNN
 	1    3350 3400
@@
 F 0 "R4" H 4620 4545 50  0000 L CNN
 F 1 "1K" H 4620 4455 50  0000 L CNN
-F 2 "" V 4480 4500 50  0001 C CNN
+F 2 "Resistor_SMD:R_0603_1608Metric_Pad0.98x0.95mm_HandSolder" V 4480 4500 50  0001 C CNN
 F 3 "~" H 4550 4500 50  0001 C CNN
 	1    4550 4500
@@
 F 0 "R2" H 3420 4445 50  0000 L CNN
 F 1 "10k" H 3420 4355 50  0000 L CNN
-F 2 "" V 3280 4400 50  0001 C CNN
+F 2 "Resistor_SMD:R_0603_1608Metric_Pad0.98x0.95mm_HandSolder" V 3280 4400 50  0001 C CNN
 F 3 "~" H 3350 4400 50  0001 C CNN
 	1    3350 4400
@@
 F 0 "TH1" H 6937 4346 50  0000 L CNN
 F 1 "SIM_NTC_10K_1" H 6937 4255 50  0000 L CNN
-F 2 "" H 6750 4350 50  0001 C CNN
+F 2 "Resistor_SMD:R_0805_2012Metric_Pad1.20x1.40mm_HandSolder" H 6750 4350 50  0001 C CNN
 F 3 "~" H 6750 4350 50  0001 C CNN
 F 4 "X" H 6750 4300 50  0001 C CNN "Spice_Primitive"
@@
 Wire Wire Line
 	8050 3900 8050 4000
-Wire Wire Line
-	8050 4600 8050 4700
-Wire Wire Line
-	8050 4700 7450 4700
-Wire Wire Line
-	6850 4700 6850 4550
-Wire Wire Line
-	7450 4700 7450 4850
-Connection ~ 7450 4700
-Wire Wire Line
-	7450 4700 6850 4700
+Text Label 7350 3900 0    50   ~ 0
+vcont
+Wire Wire Line
+	6750 2900 6750 3250
+Wire Wire Line
+	6750 3850 6750 3550
+Wire Wire Line
+	6750 3850 6750 4050
+Connection ~ 6750 3850
+Wire Wire Line
+	6750 4550 6750 4850
+$Comp
+L Device:Q_PMOS_GDS Q3
+U 1 1 606E0DAA
+P 8850 3000
+F 0 "Q3" V 9192 3000 50  0000 C CNN
+F 1 "FDD306P" V 9101 3000 50  0000 C CNN
+F 2 "Package_TO_SOT_SMD:TO-252-3_TabPin2" H 9050 3100 50  0001 C CNN
+F 3 "~" H 8850 3000 50  0001 C CNN
+F 4 "X" H 8850 3000 50  0001 C CNN "Spice_Primitive"
+F 5 "FDD306P" H 8850 3000 50  0001 C CNN "Spice_Model"
+F 6 "Y" H 8850 3000 50  0001 C CNN "Spice_Netlist_Enabled"
+F 7 "./FDD306P.lib" H 8850 3000 50  0001 C CNN "Spice_Lib_File"
+F 8 "2 1 3" H 8850 3000 50  0001 C CNN "Spice_Node_Sequence"
+	1    8850 3000
+	0    1    -1   0
+$EndComp
+Wire Wire Line
+	6750 2900 8650 2900
+Connection ~ 6750 2900
+Wire Wire Line
+	9050 2900 9200 2900
+Wire Wire Line
+	9800 2900 9800 3450
+$Comp
+L Device:R R6
+U 1 1 606F8AF7
+P 9800 3600
+F 0 "R6" H 9870 3646 50  0000 L CNN
+F 1 "5" H 9870 3555 50  0000 L CNN
+F 2 "" V 9730 3600 50  0001 C CNN
+F 3 "~" H 9800 3600 50  0001 C CNN
+	1    9800 3600
+	1    0    0    -1
+$EndComp
 $Comp
 L pspice:0 #GND02
 U 1 1 6066B092
-P 7450 4850
-F 0 "#GND02" H 7450 4750 50  0001 C CNN
-F 1 "0" H 7450 4939 50  0000 C CNN
-F 2 "" H 7450 4850 50  0001 C CNN
-F 3 "~" H 7450 4850 50  0001 C CNN
-	1    7450 4850
-	1    0    0    -1
-$EndComp
-Text Label 7350 3900 0    50   ~ 0
-vcont
-Wire Wire Line
-	6750 2900 6750 3250
-Wire Wire Line
-	6750 3850 6750 3550
-Wire Wire Line
-	6750 3850 6750 4050
-Connection ~ 6750 3850
-Wire Wire Line
-	6750 4550 6750 4850
+P 7450 4750
+F 0 "#GND02" H 7450 4650 50  0001 C CNN
+F 1 "0" H 7450 4839 50  0000 C CNN
+F 2 "" H 7450 4750 50  0001 C CNN
+F 3 "~" H 7450 4750 50  0001 C CNN
+	1    7450 4750
+	1    0    0    -1
+$EndComp
+Wire Wire Line
+	6850 4600 7450 4600
+Wire Wire Line
+	6850 4600 6850 4550
+Wire Wire Line
+	7450 4600 7450 4750
+Connection ~ 7450 4600
+Wire Wire Line
+	7450 4600 8050 4600
+Wire Wire Line
+	6750 4850 9800 4850
+Wire Wire Line
+	9800 4850 9800 3750
+Connection ~ 6750 4850
+Wire Wire Line
+	8850 3200 8850 3500
+Wire Wire Line
+	8850 3500 8500 3500
+Text Label 7550 3500 0    50   ~ 0
+VD1
+Text Label 9800 2900 0    50   ~ 0
+vload
+$Comp
+L Device:C C2
+U 1 1 60757828
+P 10400 3800
+F 0 "C2" H 10515 3846 50  0000 L CNN
+F 1 "1uF" H 10515 3755 50  0000 L CNN
+F 2 "Capacitor_SMD:C_0805_2012Metric_Pad1.18x1.45mm_HandSolder" H 10438 3650 50  0001 C CNN
+F 3 "~" H 10400 3800 50  0001 C CNN
+	1    10400 3800
+	1    0    0    -1
+$EndComp
+Wire Wire Line
+	10400 3650 10400 2900
+Wire Wire Line
+	10400 2900 9800 2900
+Connection ~ 9800 2900
+Wire Wire Line
+	10400 3950 10400 4850
+Wire Wire Line
+	10400 4850 9800 4850
+Connection ~ 9800 4850
+$Comp
+L Device:C C1
+U 1 1 6076DAA7
+P 9200 3200
+F 0 "C1" H 9315 3246 50  0000 L CNN
+F 1 "30nF" H 9315 3155 50  0000 L CNN
+F 2 "Capacitor_SMD:C_0201_0603Metric_Pad0.64x0.40mm_HandSolder" H 9238 3050 50  0001 C CNN
+F 3 "~" H 9200 3200 50  0001 C CNN
+	1    9200 3200
+	1    0    0    -1
+$EndComp
+Wire Wire Line
+	9200 3050 9200 2900
+Connection ~ 9200 2900
+Wire Wire Line
+	9200 2900 9800 2900
+Wire Wire Line
+	9200 3350 9200 3500
+Wire Wire Line
+	9200 3500 8850 3500
+Connection ~ 8850 3500
+$Comp
+L Device:R R10
+U 1 1 607712E1
+P 8350 3500
+F 0 "R10" V 8143 3500 50  0000 C CNN
+F 1 "1k" V 8234 3500 50  0000 C CNN
+F 2 "Resistor_SMD:R_0603_1608Metric_Pad0.98x0.95mm_HandSolder" V 8280 3500 50  0001 C CNN
+F 3 "~" H 8350 3500 50  0001 C CNN
+	1    8350 3500
+	0    1    1    0
+$EndComp
+Wire Wire Line
+	8200 3500 7550 3500
 $EndSCHEMATC

Commit message: Tuning simulation to change on/off temperature. Then making the resulting changes to BoM
Parts:
- R1, R7: value 6.6k -> 62k
- R2: value 10k -> 100k
- R8, R9: value 20k -> 200k
Other:
- note added: "Turn on/off at -25 C\n"
Changed lines of the file:
@@
 P 6750 3400
 F 0 "R7" H 6820 3445 50  0000 L CNN
-F 1 "6.6k" H 6820 3355 50  0000 L CNN
+F 1 "62k" H 6820 3355 50  0000 L CNN
 F 2 "Resistor_SMD:R_0603_1608Metric_Pad0.98x0.95mm_HandSolder" V 6680 3400 50  0001 C CNN
 F 3 "~" H 6750 3400 50  0001 C CNN
@@
 P 4900 3450
 F 0 "R9" V 5106 3450 50  0000 C CNN
-F 1 "20k" V 5015 3450 50  0000 C CNN
+F 1 "200k" V 5015 3450 50  0000 C CNN
 F 2 "Resistor_SMD:R_0603_1608Metric_Pad0.98x0.95mm_HandSolder" V 4830 3450 50  0001 C CNN
 F 3 "~" H 4900 3450 50  0001 C CNN
@@
 P 4300 3600
 F 0 "R8" V 4400 3600 50  0000 C CNN
-F 1 "20k" V 4200 3600 50  0000 C CNN
+F 1 "200k" V 4200 3600 50  0000 C CNN
 F 2 "Resistor_SMD:R_0603_1608Metric_Pad0.98x0.95mm_HandSolder" V 4230 3600 50  0001 C CNN
 F 3 "~" H 4300 3600 50  0001 C CNN
@@
 P 3350 3400
 F 0 "R1" H 3420 3445 50  0000 L CNN
-F 1 "6.6k" H 3420 3355 50  0000 L CNN
+F 1 "62k" H 3420 3355 50  0000 L CNN
 F 2 "Resistor_SMD:R_0603_1608Metric_Pad0.98x0.95mm_HandSolder" V 3280 3400 50  0001 C CNN
 F 3 "~" H 3350 3400 50  0001 C CNN
@@
 P 3350 4400
 F 0 "R2" H 3420 4445 50  0000 L CNN
-F 1 "10k" H 3420 4355 50  0000 L CNN
+F 1 "100k" H 3420 4355 50  0000 L CNN
 F 2 "Resistor_SMD:R_0603_1608Metric_Pad0.98x0.95mm_HandSolder" V 3280 4400 50  0001 C CNN
 F 3 "~" H 3350 4400 50  0001 C CNN
@@
 Wire Wire Line
 	8200 3500 7550 3500
+Text Notes 2500 5450 0    50   ~ 0
+Turn on/off at -25 C\n
 $EndSCHEMATC

Commit message: Changed mosfet from bss127s --> irlml2402 (which has lower threshold voltage and higher transconductance
Parts:
- removed Q1, Q2: BSS127S, Package_TO_SOT_SMD:SOT-23, symbol Transistor_FET:BSS127S
- added Q1, Q2: IRLML2402TR, Package_TO_SOT_SMD:SOT-23, symbol kicad_cryosub_simlib:IRLML2402TR
- R1, R7: value 62k -> 100k
Connections:
- net VD1: now also Q1.3 (D)
- net vd2: now also Q2.3 (D)
- net vg1: now also Q1.1 (G)
- net vg2: now also Q2.1 (G)
- net vs: now also Q1.2 (S), Q2.2 (S)
Changed lines of the file:
@@
 P 6750 3400
 F 0 "R7" H 6820 3445 50  0000 L CNN
-F 1 "62k" H 6820 3355 50  0000 L CNN
+F 1 "100k" H 6820 3355 50  0000 L CNN
 F 2 "Resistor_SMD:R_0603_1608Metric_Pad0.98x0.95mm_HandSolder" V 6680 3400 50  0001 C CNN
 F 3 "~" H 6750 3400 50  0001 C CNN
@@
 Wire Wire Line
 	4450 3600 5800 3600
-$Comp
-L Transistor_FET:BSS127S Q2
-U 1 1 605C1A8E
-P 5350 3850
-F 0 "Q2" H 5555 3895 50  0000 L CNN
-F 1 "BSS127S" H 5555 3805 50  0000 L CNN
-F 2 "Package_TO_SOT_SMD:SOT-23" H 5550 3775 50  0001 L CIN
-F 3 "http://www.diodes.com/assets/Datasheets/BSS127.pdf" H 5350 3850 50  0001 L CNN
-F 4 "X" H 5350 3850 50  0001 C CNN "Spice_Primitive"
-F 5 "BSS127_L0" H 5350 3850 50  0001 C CNN "Spice_Model"
-F 6 "Y" H 5350 3850 50  0001 C CNN "Spice_Netlist_Enabled"
-F 7 "./IFX-Power_OptiMOS_N-channel_small_signal_MOSFET_240V_250V_400V_600V_Spice-web.lib" H 5350 3850 50  0001 C CNN "Spice_Lib_File"
-F 8 "3 1 2" H 5350 3850 50  0001 C CNN "Spice_Node_Sequence"
-	1    5350 3850
-	-1   0    0    -1
-$EndComp
 Connection ~ 4550 4850
 Wire Wire Line
@@
 Connection ~ 5250 3450
 $Comp
-L Transistor_FET:BSS127S Q1
-U 1 1 605BE7F9
-P 3850 3850
-F 0 "Q1" H 4055 3895 50  0000 L CNN
-F 1 "BSS127S" H 4055 3805 50  0000 L CNN
-F 2 "Package_TO_SOT_SMD:SOT-23" H 4050 3775 50  0001 L CIN
-F 3 "http://www.diodes.com/assets/Datasheets/BSS127.pdf" H 3850 3850 50  0001 L CNN
-F 4 "X" H 3850 3850 50  0001 C CNN "Spice_Primitive"
-F 5 "BSS127_L0" H 3850 3850 50  0001 C CNN "Spice_Model"
-F 6 "Y" H 3850 3850 50  0001 C CNN "Spice_Netlist_Enabled"
-F 7 "./IFX-Power_OptiMOS_N-channel_small_signal_MOSFET_240V_250V_400V_600V_Spice-web.lib" H 3850 3850 50  0001 C CNN "Spice_Lib_File"
-F 8 "3 1 2 " H 3850 3850 50  0001 C CNN "Spice_Node_Sequence"
-	1    3850 3850
-	1    0    0    -1
-$EndComp
-$Comp
 L Device:R R5
 U 1 1 605937CE
@@
 P 3350 3400
 F 0 "R1" H 3420 3445 50  0000 L CNN
-F 1 "62k" H 3420 3355 50  0000 L CNN
+F 1 "100k" H 3420 3355 50  0000 L CNN
 F 2 "Resistor_SMD:R_0603_1608Metric_Pad0.98x0.95mm_HandSolder" V 3280 3400 50  0001 C CNN
 F 3 "~" H 3350 3400 50  0001 C CNN
@@
 Text Notes 2500 5450 0    50   ~ 0
 Turn on/off at -25 C\n
+$Comp
+L kicad_cryosub_simlib:IRLML2402TR Q1
+U 1 1 60A27F5B
+P 3850 3850
+F 0 "Q1" H 4054 4123 50  0000 L CNN
+F 1 "IRLML2402TR" H 4054 4032 50  0000 L CNN
+F 2 "Package_TO_SOT_SMD:SOT-23" H 4050 3775 50  0001 L CIN
+F 3 "https://docs.rs-online.com/c4e5/0900766b80afb7ed.pdf" H 3850 3850 50  0001 L CNN
+F 4 "X" H 4054 3941 50  0000 L CNN "Spice_Primitive"
+F 5 "irlml2402" H 4054 3850 50  0000 L CNN "Spice_Model"
+F 6 "Y" H 4054 3759 50  0000 L CNN "Spice_Netlist_Enabled"
+F 7 "3 1 2" H 4054 3668 50  0000 L CNN "Spice_Node_Sequence"
+F 8 "irlml2402.lib" H 4054 3577 50  0000 L CNN "Spice_Lib_File"
+	1    3850 3850
+	1    0    0    -1
+$EndComp
+$Comp
+L kicad_cryosub_simlib:IRLML2402TR Q2
+U 1 1 60A2FA09
+P 5350 3850
+F 0 "Q2" H 5555 4123 50  0000 L CNN
+F 1 "IRLML2402TR" H 5555 4032 50  0000 L CNN
+F 2 "Package_TO_SOT_SMD:SOT-23" H 5550 3775 50  0001 L CIN
+F 3 "https://docs.rs-online.com/c4e5/0900766b80afb7ed.pdf" H 5350 3850 50  0001 L CNN
+F 4 "X" H 5555 3941 50  0000 L CNN "Spice_Primitive"
+F 5 "irlml2402" H 5555 3850 50  0000 L CNN "Spice_Model"
+F 6 "Y" H 5555 3759 50  0000 L CNN "Spice_Netlist_Enabled"
+F 7 "3 1 2" H 5555 3668 50  0000 L CNN "Spice_Node_Sequence"
+F 8 "irlml2402.lib" H 5555 3577 50  0000 L CNN "Spice_Lib_File"
+	1    5350 3850
+	-1   0    0    -1
+$EndComp
 $EndSCHEMATC
