File: hardware/uob-hep-pc068a-cryosub/cryosub_top_v01/onWhenWarm.sch (KiCad schematic (older format))
At the start: 16 parts, among them Q1 BSS127S, Q2 BSS127S, Q3 FDD306P

Commit message: Tuning simulation to change on/off temperature. Then making the resulting changes to BoM
Parts:
- R1, R8: value 6.6k -> 62k
- R4, R6: value 10k -> 200k
Other:
- note added: ""On when warm"\nTurn on at -23 C when warming up\nTurn off at -31 C when cooling down"
Changed lines of the file:
@@
 P 6750 3400
 F 0 "R8" H 6820 3445 50  0000 L CNN
-F 1 "6.6k" H 6820 3355 50  0000 L CNN
+F 1 "62k" H 6820 3355 50  0000 L CNN
 F 2 "Resistor_SMD:R_0603_1608Metric_Pad0.98x0.95mm_HandSolder" V 6680 3400 50  0001 C CNN
 F 3 "~" H 6750 3400 50  0001 C CNN
@@
 P 4900 3450
 F 0 "R6" V 5106 3450 50  0000 C CNN
-F 1 "10k" V 5015 3450 50  0000 C CNN
+F 1 "200k" V 5015 3450 50  0000 C CNN
 F 2 "Resistor_SMD:R_0603_1608Metric_Pad0.98x0.95mm_HandSolder" V 4830 3450 50  0001 C CNN
 F 3 "~" H 4900 3450 50  0001 C CNN
@@
 P 4300 3600
 F 0 "R4" V 4400 3600 50  0000 C CNN
-F 1 "10k" V 4200 3600 50  0000 C CNN
+F 1 "200k" V 4200 3600 50  0000 C CNN
 F 2 "Resistor_SMD:R_0603_1608Metric_Pad0.98x0.95mm_HandSolder" V 4230 3600 50  0001 C CNN
 F 3 "~" H 4300 3600 50  0001 C CNN
@@
 P 3350 3400
 F 0 "R1" H 3420 3445 50  0000 L CNN
-F 1 "6.6k" H 3420 3355 50  0000 L CNN
+F 1 "62k" H 3420 3355 50  0000 L CNN
 F 2 "Resistor_SMD:R_0603_1608Metric_Pad0.98x0.95mm_HandSolder" V 3280 3400 50  0001 C CNN
 F 3 "~" H 3350 3400 50  0001 C CNN
@@
 Text Notes 8000 3850 0    50   ~ 0
 RC to slow turn-on of load switch\nand reduce inrush current
+Text Notes 7150 6950 0    50   ~ 0
+"On when warm"\nTurn on at -23 C when warming up\nTurn off at -31 C when cooling down
 $EndSCHEMATC

Commit message: Updated BoM, correctly this time I hope, to update resistor values for correct set-points
Parts:
- R2: value 10k -> 100k
Changed lines of the file:
@@
 P 3350 4400
 F 0 "R2" H 3420 4445 50  0000 L CNN
-F 1 "10k" H 3420 4355 50  0000 L CNN
+F 1 "100k" H 3420 4355 50  0000 L CNN
 F 2 "Resistor_SMD:R_0603_1608Metric_Pad0.98x0.95mm_HandSolder" V 3280 4400 50  0001 C CNN
 F 3 "~" H 3350 4400 50  0001 C CNN

Commit message: Changed mosfet from bss127s --> irlml2402 (which has lower threshold voltage and higher transconductance
Parts:
- Q1, Q2: value BSS127S -> IRLML2402TR
- R1, R8: value 62k -> 100k
Changed lines of the file:
@@
 P 6750 3400
 F 0 "R8" H 6820 3445 50  0000 L CNN
-F 1 "62k" H 6820 3355 50  0000 L CNN
+F 1 "100k" H 6820 3355 50  0000 L CNN
 F 2 "Resistor_SMD:R_0603_1608Metric_Pad0.98x0.95mm_HandSolder" V 6680 3400 50  0001 C CNN
 F 3 "~" H 6750 3400 50  0001 C CNN
@@
 P 5350 3850
 F 0 "Q2" H 5555 3895 50  0000 L CNN
-F 1 "BSS127S" H 5555 3805 50  0000 L CNN
+F 1 "IRLML2402TR" H 5555 3805 50  0000 L CNN
 F 2 "Package_TO_SOT_SMD:SOT-23" H 5550 3775 50  0001 L CIN
 F 3 "http://www.diodes.com/assets/Datasheets/BSS127.pdf" H 5350 3850 50  0001 L CNN
@@
 P 3850 3850
 F 0 "Q1" H 4055 3895 50  0000 L CNN
-F 1 "BSS127S" H 4055 3805 50  0000 L CNN
+F 1 "IRLML2402TR" H 4055 3805 50  0000 L CNN
 F 2 "Package_TO_SOT_SMD:SOT-23" H 4050 3775 50  0001 L CIN
 F 3 "http://www.diodes.com/assets/Datasheets/BSS127.pdf" H 3850 3850 50  0001 L CNN
@@
 P 3350 3400
 F 0 "R1" H 3420 3445 50  0000 L CNN
-F 1 "62k" H 3420 3355 50  0000 L CNN
+F 1 "100k" H 3420 3355 50  0000 L CNN
 F 2 "Resistor_SMD:R_0603_1608Metric_Pad0.98x0.95mm_HandSolder" V 3280 3400 50  0001 C CNN
 F 3 "~" H 3350 3400 50  0001 C CNN
