File: hardware/uob-hep-pc068a-cryosub/cryosub_power_converter_top_v02/cryosub_power_converter_top_v02.sch (KiCad schematic (older format))
At the start: 12 parts, among them J1 Conn_01x02_Male, J2 Conn_02x05_Odd_Even, J3 Conn_01x02_Male, U1 LT3042xMSE

Commit message: Comitting version with 5V-->48V DC-DC converter
Changed lines of the file:
@@
 $Descr A4 11693 8268
 encoding utf-8
-Sheet 1 3
+Sheet 1 4
 Title ""
 Date ""
@@
 Wire Wire Line
 	1450 2750 2250 2750
+$Sheet
+S 5250 900  900  600
+U 6196D499
+F0 "sipm_dcdc" 50
+F1 "sipm_dcdc.sch" 50
+$EndSheet
+Text HLabel 5250 1050 0    50   Input ~ 0
+vin
+Text HLabel 6150 1050 0    50   Output ~ 0
+vout
+Text HLabel 5250 1250 0    50   Input ~ 0
+enable
+Text HLabel 5250 1450 0    50   BiDi ~ 0
+gnd
 $EndSCHEMATC
