File: hardware/uob-hep-pc068a-cryosub/cryosub_power_converter_top_v02/dc_dc.sch (KiCad schematic (older format))
At the start: 9 parts

Commit message: Comitting version with 5V-->48V DC-DC converter
Parts:
- L1, L2: value 4.7uH -> 1.0uH
Changed lines of the file:
@@
 $Descr A4 11693 8268
 encoding utf-8
-Sheet 3 3
+Sheet 3 4
 Title ""
 Date ""
@@
 P 4100 3050
 F 0 "L1" V 3919 3050 50  0000 C CNN
-F 1 "4.7uH" V 4010 3050 50  0000 C CNN
+F 1 "1.0uH" V 4010 3050 50  0000 C CNN
 F 2 "Inductor_SMD:L_0603_1608Metric_Pad1.05x0.95mm_HandSolder" H 4100 3050 50  0001 C CNN
 F 3 "~" H 4100 3050 50  0001 C CNN
@@
 P 7800 3050
 F 0 "L2" V 7619 3050 50  0000 C CNN
-F 1 "4.7uH" V 7710 3050 50  0000 C CNN
+F 1 "1.0uH" V 7710 3050 50  0000 C CNN
 F 2 "Inductor_SMD:L_0603_1608Metric_Pad1.05x0.95mm_HandSolder" H 7800 3050 50  0001 C CNN
 F 3 "~" H 7800 3050 50  0001 C CNN
