File: hardware/uob-hep-pc068a-cryosub/cryosub_power_converter_top_v03/dc_dc.kicad_sch (KiCad schematic)
At the start: 13 parts

Commit message: Tweaked layout to remove DRCs (mainly silk) removed duplicate D1
Parts:
- R13: footprint Resistor_SMD:R_0402_1005Metric -> (none)
Changed lines of the file:
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@@
       (effects (font (size 1.27 1.27)) (justify left))
     )
-    (property "Footprint" "Resistor_SMD:R_0402_1005Metric" (id 2) (at 88.9 95.758 90)
+    (property "Footprint" "" (id 2) (at 88.9 95.758 90)
       (effects (font (size 1.27 1.27)) hide)
     )

Commit message: Replacing FDD306 with SiS407
Parts:
- C12: value (none) -> 22uF; footprint (none) -> Capacitor_SMD:C_0805_2012Metric_Pad1.18x1.45mm_HandSolder
- R13: footprint (none) -> Resistor_SMD:R_0603_1608Metric
- U2: value (none) -> LTC3129IMSE-1-PBF
Changed lines of the file:
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@@
       (effects (font (size 1.27 1.27)) (justify left))
     )
-    (property "Value" "" (id 1) (at 195.961 86.233 0)
+    (property "Value" "22uF" (id 1) (at 195.961 86.233 0)
       (effects (font (size 1.27 1.27)) (justify left))
     )
-    (property "Footprint" "" (id 2) (at 194.0052 88.9 0)
+    (property "Footprint" "Capacitor_SMD:C_0805_2012Metric_Pad1.18x1.45mm_HandSolder" (id 2) (at 194.0052 88.9 0)
       (effects (font (size 1.27 1.27)) hide)
     )
@@
       (effects (font (size 1.524 1.524)))
     )
-    (property "Value" "" (id 1) (at 119.38 63.9826 0)
+    (property "Value" "LTC3129IMSE-1-PBF" (id 1) (at 119.38 63.9826 0)
       (effects (font (size 1.524 1.524)))
     )
@@
       (effects (font (size 1.27 1.27)) (justify left))
     )
-    (property "Footprint" "" (id 2) (at 88.9 95.758 90)
+    (property "Footprint" "Resistor_SMD:R_0603_1608Metric" (id 2) (at 88.9 95.758 90)
       (effects (font (size 1.27 1.27)) hide)
     )
